File: GMA1_SOM/DISPLAY.kicad_sch (KiCad schematic)
At the start: 0 parts

Commit message: add display and ram
Parts:
- added Q1, Q10, Q2, Q3, Q4, Q5, Q6, Q7, Q8, Q9: BSS138, Package_TO_SOT_SMD:SOT-23, symbol Transistor_FET:BSS138
- added R26, R27, R28, R29, R30, R31, R32, R33, R34, R35, R36, R37, R38, R39, R40, R41, R42, R43: R_US, symbol Device:R_US
- added U8: HDSM-543B, Display:HDSM-541B_HDSM-543B, symbol Display_Character:HDSM-543B
Connections:
- new net: Q2.1 (G), R28.2
- new net: Q10.1 (G), R42.2
- new net: Q10.2 (S), U8.9 (B)
- new net: Q10.3 (D), R43.1
- new net: Q5.3 (D), R33.1
- new net: Q6.3 (D), R35.1
- new net: Q6.1 (G), R34.2
- new net: Q3.1 (G), R29.2
- new net: Q5.1 (G), R32.2
- new net: Q7.1 (G), R36.2
- new net: Q1.3 (D), R27.1
- new net: Q9.1 (G), R40.2
- new net: Q7.2 (S), U8.6 (D)
- new net: Q7.3 (D), R37.1
- new net: Q1.1 (G), R26.2
- new net: Q4.3 (D), R31.1
- new net: Q8.1 (G), R38.2
- new net: Q8.2 (S), U8.7 (E)
- new net: Q8.3 (D), R39.1
- new net: Q4.1 (G), R30.2
- new net: Q6.2 (S), U8.4 (F)
- new net: Q1.2 (S), U8.1 (G)
- new net: Q2.2 (S), U8.10 (CC_DIG1)
- new net: Q9.3 (D), R41.1
- new net: Q5.2 (S), U8.3 (A)
- new net: Q4.2 (S), U8.2 (DP)
- new net: Q3.2 (S), U8.5 (CC_DIG2)
- new net: Q9.2 (S), U8.8 (C)
- new net +3V3: R27.2, R31.2, R33.2, R35.2, R37.2, R39.2, R41.2, R43.2
- new net A: R32.1
- new net B: R42.1
- new net C: R40.1
- new net CC1: R28.1
- new net CC2: R29.1
- new net D: R36.1
- new net DP: R30.1
- new net E: R38.1
- new net F: R34.1
- new net G: R26.1
- new net GND: Q2.3 (D), Q3.3 (D)
