File: GMA1_SOM/FPGA.kicad_sch (KiCad schematic)
At the start: 2 parts, among them J2 SODIMM-200_Split, U1 CCGM1A1

Commit message: add display and ram
Connections:
- net DQ0: now reaches U1.G15 (IO_EA_B8)
- net CLK: now reaches U1.G16 (IO_EA_A8)
- net ~{ADV}: now reaches U1.G17 (IO_EA_B7)
- net ~{WE}: now reaches U1.G18 (IO_EA_A7)
- net ~{CE}: now reaches U1.H15 (IO_EA_B6)
- net ~{UB}: now reaches U1.H16 (IO_EA_A6)
- net ~{LB}: now reaches U1.J15 (IO_EA_B5)
- net CRE: now reaches U1.J16 (IO_EA_A5)
- net ~{OE}: now reaches U1.J17 (IO_EA_B4)
- net WAIT0: now reaches U1.J18 (IO_EA_A4)
- net WAIT1: now reaches U1.K15 (IO_EA_B3)
- net IO_WB_A3: now reaches U1.L1 (IO_WB_A3)
- net IO_WB_B3: now reaches U1.L2 (IO_WB_B3)
- net IO_WB_A2: now reaches U1.L3 (IO_WB_A2)
- net IO_WB_B2: now reaches U1.L4 (IO_WB_B2)
- net A5: now reaches U1.A11 (IO_NB_B2)
- net A9: now reaches U1.A12 (IO_NB_B4)
- net A15: now reaches U1.A14 (IO_NB_B7)
- net DQ1: now reaches U1.A3 (IO_NA_A0)
- net DQ3: now reaches U1.A4 (IO_NA_A1)
- net DQ9: now reaches U1.A6 (IO_NA_A4)
- net DQ15: now reaches U1.A8 (IO_NA_A7)
- net A1: now reaches U1.A9 (IO_NB_B0)
- net A4: now reaches U1.B11 (IO_NB_A2)
- net A8: now reaches U1.B12 (IO_NB_A4)
- net A14: now reaches U1.B14 (IO_NB_A7)
- net DQ2: now reaches U1.B3 (IO_NA_B0)
- net DQ4: now reaches U1.B4 (IO_NA_B1)
- net DQ5: now reaches U1.B5 (IO_NA_A2)
- net DQ10: now reaches U1.B6 (IO_NA_B4)
- net A20: now reaches U1.B8 (IO_NA_B7)
- net A0: now reaches U1.B9 (IO_NB_A0)
- net A3: now reaches U1.C10 (IO_NB_B1)
- net A7: now reaches U1.C11 (IO_NB_B3)
- net A11: now reaches U1.C12 (IO_NB_B5)
- net A13: now reaches U1.C13 (IO_NB_B6)
- net A17: now reaches U1.C14 (IO_NB_B8)
- net DQ6: now reaches U1.C5 (IO_NA_B2)
- net DQ7: now reaches U1.C6 (IO_NA_A3)
- net DQ11: now reaches U1.C7 (IO_NA_A5)
- net DQ13: now reaches U1.C8 (IO_NA_A6)
- net A19: now reaches U1.C9 (IO_NA_A8)
- net A2: now reaches U1.D10 (IO_NB_A1)
- net A6: now reaches U1.D11 (IO_NB_A3)
- net A10: now reaches U1.D12 (IO_NB_A5)
- net A12: now reaches U1.D13 (IO_NB_A6)
- net A16: now reaches U1.D14 (IO_NB_A8)
- net DQ8: now reaches U1.D6 (IO_NA_B3)
- net DQ12: now reaches U1.D7 (IO_NA_B5)
- net DQ14: now reaches U1.D8 (IO_NA_B6)
- net A18: now reaches U1.D9 (IO_NA_B8)
- net GND: now reaches U1.A1 (GND), U1.A10 (GND), U1.A13 (GND), U1.A18 (GND), U1.A7 (GND), U1.B16 (GND), U1.C1 (GND), U1.E11 (GND), U1.E13 (GND), U1.E18 (GND), U1.E5 (GND), U1.E7 (GND), U1.E9 (GND), U1.F1 (GND), U1.F10 (GND), U1.F12 (GND), U1.F14 (GND), U1.F6 (GND), U1.F8 (GND), U1.G11 (GND), U1.G13 (GND), U1.G5 (GND), U1.G7 (GND), U1.G9 (GND), U1.H10 (GND), U1.H12 (GND), U1.H14 (GND), U1.H18 (GND), U1.H6 (GND), U1.H8 (GND), U1.J1 (GND), U1.J11 (GND), U1.J13 (GND), U1.J5 (GND), U1.J7 (GND), U1.J9 (GND), U1.K10 (GND), U1.K12 (GND), U1.K14 (GND), U1.K6 (GND), U1.K8 (GND), U1.L11 (GND), U1.L13 (GND), U1.L18 (GND), U1.L5 (GND), U1.L7 (GND), U1.L9 (GND), U1.M1 (GND), U1.M10 (GND), U1.M12 (GND), U1.M16 (GND), U1.M6 (GND), U1.M8 (GND), U1.N12 (GND), U1.N17 (GND), U1.N7 (GND), U1.N9 (GND), U1.P4 (GND), U1.P7 (GND), U1.P9 (GND), U1.R12 (GND), U1.R16 (GND), U1.T11 (GND), U1.T17 (GND), U1.T4 (GND), U1.U14 (GND), U1.U15 (GND), U1.U16 (GND), U1.V1 (GND), U1.V14 (GND), U1.V16 (GND), U1.V18 (GND), U1.V6 (GND), U1.V9 (GND)
Other:
- moved on the sheet: J2B, J2D, U1A, U1B, U1C, U1D, U1F, U1G
