File: GMA1_SOM/RAM.kicad_sch (KiCad schematic)
At the start: 0 parts

Commit message: add display and ram
Parts:
- added R1, R2, R3, R4, R5, R6: 1K, symbol Device:R_US
- added R7: 12K1, symbol Device:R_US
- added U3: IS66WVC2M16EALL-7010BLI, Project_Library:BGA-54_6x9_6.0x8.0mm, symbol Project_Library:IS66WVC2M16EALL-7010BLI
Connections:
- new net +1V8: R1.2, R2.2, R3.2, R4.2, R5.2, R6.2, U3.D6 (VDD), U3.E1 (VDDQ)
- new net A0: U3.A3 (A0)
- new net A1: U3.A4 (A1)
- new net A10: U3.H4 (A10)
- new net A11: U3.H5 (A11)
- new net A12: U3.G3 (A12)
- new net A13: U3.G4 (A13)
- new net A14: U3.F3 (A14)
- new net A15: U3.F4 (A15)
- new net A16: U3.E4 (A16)
- new net A17: U3.D3 (A17)
- new net A18: U3.H1 (A18)
- new net A19: U3.G2 (A19)
- new net A2: U3.A5 (A2)
- new net A20: U3.H6 (A20)
- new net A3: U3.B3 (A3)
- new net A4: U3.B4 (A4)
- new net A5: U3.C3 (A5)
- new net A6: U3.C4 (A6)
- new net A7: U3.D4 (A7)
- new net A8: U3.H2 (A8)
- new net A9: U3.H3 (A9)
- new net CLK: U3.J2 (CLK)
- new net CRE: R7.2, U3.A6 (CRE)
- new net DQ0: U3.B6 (DQ0)
- new net DQ1: U3.C5 (DQ1)
- new net DQ10: U3.C2 (DQ10)
- new net DQ11: U3.D2 (DQ11)
- new net DQ12: U3.E2 (DQ12)
- new net DQ13: U3.F2 (DQ13)
- new net DQ14: U3.F1 (DQ14)
- new net DQ15: U3.G1 (DQ15)
- new net DQ2: U3.C6 (DQ2)
- new net DQ3: U3.D5 (DQ3)
- new net DQ4: U3.E5 (DQ4)
- new net DQ5: U3.F5 (DQ5)
- new net DQ6: U3.F6 (DQ6)
- new net DQ7: U3.G6 (DQ7)
- new net DQ8: U3.B1 (DQ8)
- new net DQ9: U3.C1 (DQ9)
- new net GND: R7.1, U3.D1 (VSSQ), U3.E6 (VSS)
- new net WAIT: U3.J1 (WAIT)
- new net ~{ADV}: R1.1, U3.J3 (~{ADV})
- new net ~{CE}: R3.1, U3.B5 (~{CE})
- new net ~{LB}: R5.1, U3.A1 (~{LB})
- new net ~{OE}: R6.1, U3.A2 (~{OE})
- new net ~{UB}: R4.1, U3.B2 (~{UB})
- new net ~{WE}: R2.1, U3.G5 (~{WE})
